Commit message: add gazebo simulations and obstacles

File: description/robot.urdf.xacro (robot description, xacro)
@@ -1,4 +1,5 @@
 <?xml version="1.0"?>
 <robot xmlns:xacro="http://www.ros.org/wiki/xacro"  name="robot">
-    <xacro:include filename="robo_core.xacro" />
+    <xacro:include filename="robot_core.xacro" />
+    <xacro:include filename="gazebo_control.xacro" />
 </robot>

File: description/robot_core.xacro (robot description, xacro)
@@ -1,5 +1,5 @@
 <?xml version="1.0"?>
-<robot xmlns:xacro="http://www.ros.org/wiki/xacro">
-    <xacro:include filename="inertial_macros.xacro" />
+<robot xmlns:xacro="http://www.ros.org/wiki/xacro" >
+    <xacro:include filename="inertial_macros.xacro"/>
     <material name="white">
         <color rgba="1 1 1 1" />
@@ -14,8 +14,8 @@
         <color rgba="0 0 0 1"/>
     </material>
-<!-- BASE LINK -->
+    <!-- BASE LINK -->
     <link name="base_link">
     </link>
-<!-- CHASSIS LINK -->
+    <!-- CHASSIS LINK -->
     <joint name="chassis_joint" type="fixed">
         <parent link="base_link"/>
@@ -25,21 +25,24 @@
     <link name="chassis">
         <visual>
-            <origin xyz="0.15 0 0.075" />
+            <origin xyz="0.15 0 0.075"/>
             <geometry>
-                <box size="0.3 0.3 0.15" />
+                <box size="0.3 0.3 0.15"/>
             </geometry>
-            <material name="white" />
+            <material name="white"/>
         </visual>
         <collision>
-            <origin xyz="0.15 0 0.075" />
+            <origin xyz="0.15 0 0.075"/>
             <geometry>
-                <box size="0.3 0.3 0.15" />
+                <box size="0.3 0.3 0.15"/>
             </geometry>
         </collision>
         <xacro:inertial_box mass="0.5" x="0.3" y="0.3" z="0.15">
-            <orgin xyz="0.5 0 0.075" rpy="0 0 0" />
+            <origin xyz="0.15 0 0.075" rpy="0 0 0"/>
         </xacro:inertial_box>
     </link>
-<!-- LEFT WHEEL LINK -->
+    <gazebo reference="chassis">
+        <material>Gazebo/White</material>
+    </gazebo>
+    <!-- LEFT WHEEL LINK -->
     <joint name="left_wheel_joint" type="continuous">
         <parent link="base_link"/>
@@ -64,5 +67,8 @@
         </xacro:inertial_cylinder>
     </link>
-<!-- Right WHEEL LINK -->
+    <gazebo reference="left_wheel">
+        <material>Gazebo/Blue</material>
+    </gazebo>
+    <!-- RIGHT WHEEL LINK -->
     <joint name="right_wheel_joint" type="continuous">
         <parent link="base_link"/>
@@ -87,5 +93,8 @@
         </xacro:inertial_cylinder>
     </link>
-<!-- CASTER WHEEL LINK -->
+    <gazebo reference="right_wheel">
+        <material>Gazebo/Blue</material>
+    </gazebo>
+    <!-- CASTER WHEEL LINK -->
     <joint name="caster_wheel_joint" type="fixed">
         <parent link="chassis"/>
@@ -109,3 +118,8 @@
         </xacro:inertial_sphere>
     </link>
+    <gazebo reference="caster_wheel">
+        <material>Gazebo/Black</material>
+        <mu1 value="0.001"/>
+        <mu2 value="0.001"/>
+    </gazebo>
 </robot>
